File: breakout_heltec_wifi_lora_32.kicad_pcb (KiCad board)
At the start: 2 copper layers, 100 x 100 mm, 9 parts, among them J2 Screw_Terminal_01x18, J3 Screw_Terminal_01x18, U2 Logo AgroTechLab, U3 Logo CC-BY-SA

Commit message: feat: Updated PCB to v0.3.0
Routing:
- added copper zone on B.Cu, net Net-(J2-Pin_1)
Other:
- board text added: "v0.3.0"
- board text removed: "v0.2.0"
Changed lines of the file:
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@@
 	(title_block
 		(title "Breakout Board for Heltec WiFi LoRa 32")
-		(date "2025-05-31")
-		(rev "v0.2.0")
+		(date "2025-06-03")
+		(rev "v0.3.0")
 		(company "AgroTechLab (Agribusiness Technology Development Laboratory)")
 		(comment 1 "IFSC (Federal Institute of Santa Catarina)")
@@
 	)
 	(setup
+		(stackup
+			(layer "F.SilkS"
+				(type "Top Silk Screen")
+			)
+			(layer "F.Paste"
+				(type "Top Solder Paste")
+			)
+			(layer "F.Mask"
+				(type "Top Solder Mask")
+				(thickness 0.01)
+			)
+			(layer "F.Cu"
+				(type "copper")
+				(thickness 0.035)
+			)
+			(layer "dielectric 1"
+				(type "core")
+				(thickness 1.51)
+				(material "FR4")
+				(epsilon_r 4.5)
+				(loss_tangent 0.02)
+			)
+			(layer "B.Cu"
+				(type "copper")
+				(thickness 0.035)
+			)
+			(layer "B.Mask"
+				(type "Bottom Solder Mask")
+				(thickness 0.01)
+			)
+			(layer "B.Paste"
+				(type "Bottom Solder Paste")
+			)
+			(layer "B.SilkS"
+				(type "Bottom Silk Screen")
+			)
+			(copper_finish "HAL SnPb")
+			(dielectric_constraints no)
+		)
 		(pad_to_mask_clearance 0)
 		(allow_soldermask_bridges_in_footprints no)
@@
 		)
 	)
-	(gr_text "v0.2.0"
+	(gr_text "v0.3.0"
 		(at 102.66 99.86 90)
 		(layer "F.SilkS")
@@
 		(connect_pads
 			(clearance 0.5)
+		)
+		(min_thickness 0.25)
+		(filled_areas_thickness no)
+		(fill yes
+			(thermal_gap 0.5)
+			(thermal_bridge_width 0.5)
+		)
+		(polygon
+			(pts
+				(xy 96.03 45.28) (xy 195.93 45.28) (xy 195.93 145.18) (xy 96.03 145.18)
+			)
+		)
+	)
+	(zone
+		(net 13)
+		(net_name "Net-(J2-Pin_1)")
+		(layer "B.Cu")
+		(hatch edge 0.5)
+		(priority 1)
+		(connect_pads
+			(clearance 0.5)
